Commit message: Fix: проблемы с urdf-файлами после рефакторинга.

File: thor_description/urdf/thor.urdf.xacro (robot description, xacro)
@@ -1,310 +1,312 @@
 <?xml version="1.0"?>
 <robot xmlns:xacro="http://wiki.ros.org/xacro" name="$(arg name)">
-  <!-- Мировая система координат -->
-  <link name="world" />
-  <!-- ===============================================================-->
-  <!-- Робот-манипулятора, начало кинематической цепи thor_manipulator -->
-  <!-- ===============================================================-->
-  <!-- Основание робота -->
-  <joint name="base_joint" type="fixed">
-    <origin rpy="0 0 0" xyz="0 0 0"/>
-    <parent link="world"/>
-    <child link="base_link" />
-  </joint>
-  <link name="base_link">
-    <inertial>
-      <origin rpy="0 0 0" xyz="-4.6941E-06 0.054174 0.038824"/>
-      <mass value="0.7102"/>
-      <inertia ixx="0.0039943" ixy="3.697E-07" ixz="-5.7364E-08" iyy="0.0014946" iyz="-0.00036051" izz="0.0042554"/>
-    </inertial>
-    <visual>
+  <xacro:macro name="thor_robot">
+    <!-- Мировая система координат -->
+    <link name="world" />
+    <!-- ===============================================================-->
+    <!-- Робот-манипулятора, начало кинематической цепи thor_manipulator -->
+    <!-- ===============================================================-->
+    <!-- Основание робота -->
+    <joint name="base_joint" type="fixed">
       <origin rpy="0 0 0" xyz="0 0 0"/>
-      <geometry>
-        <mesh filename="file://$(find thor_description)/meshes/base.stl" scale="0.001 0.001 0.001" />
-      </geometry>
-      <material name="filament">
-        <color rgba="0.69803922 0.82352941 0.94117647 1.0"/>
-      </material>
-    </visual>
-    <collision>
-      <origin rpy="0 0 0" xyz="0 0 0"/>
-      <geometry>
-        <mesh filename="file://$(find thor_description)/meshes/base.stl" scale="0.001 0.001 0.001"/>
-      </geometry>
-    </collision>
-  </link>
-  <!-- Блок с электроникой -->
-  <joint name="box_joint" type="fixed">
-    <origin xyz="-0.1 0 0.025" rpy="0 0 0"/>
-    <parent link="base_link"/>
-    <child link="box_link"/>
-  </joint>
-  <link name="box_link">
-      <visual>
-        <geometry>
-          <box size="0.18 0.15 0.05"/>
-        </geometry>
-        <material name="filament"/>
-      </visual>
-  </link>
-  <!-- <Блок Art 1 -->
-  <link name="link_1">
-    <inertial>
-      <origin rpy="0 0 0" xyz="-0.022706 0.04294 -0.12205"/>
-      <mass value="0.88065"/>
-      <inertia ixx="0.0034" ixy="0.00042296" ixz="-0.00089231" iyy="0.0041778" iyz="0.0010848" izz="0.0027077"/>
-    </inertial>
-    <visual>
-      <origin rpy="0 0 0" xyz="0 0 0"/>
-      <geometry>
-        <mesh filename="file://$(find thor_description)/meshes/art1.stl" scale="0.001 0.001 0.001"/>
-      </geometry>
-      <material name="filament"/>
-    </visual>
-    <collision>
-      <origin rpy="0 0 0" xyz="0 0 0"/>
-      <geometry>
-        <mesh filename="file://$(find thor_description)/meshes/art1.stl" scale="0.001 0.001 0.001"/>
-      </geometry>
-    </collision>
-  </link>
-  <joint name="joint_1" type="revolute">
-    <origin xyz="0 0 0.104" rpy="0 0 0"/>
-    <parent link="base_link"/>
-    <child link="link_1"/>
-    <axis xyz="0 0 1"/>
-    <limit lower="-1.5" upper="1.5" effort="4" velocity="1.1" />
-  </joint>
-  <!-- Блок Art 2 -->
-  <link name="link_2">
-    <inertial>
-      <origin rpy="0 0 0" xyz="0.064818 -0.11189 -0.038671"/>
-      <mass value="0.57738"/>
-      <inertia ixx="0.0047312" ixy="0.0022624" ixz="0.00032144" iyy="0.0020836" iyz="-0.00056569" izz="0.0056129"/>
-    </inertial>
-    <visual>
-      <origin rpy="0 0 0" xyz="0 0 0"/>
-      <geometry>
-        <mesh filename="file://$(find thor_description)/meshes/art2.stl" scale="0.001 0.001 0.001"/>
-      </geometry>
-      <material name="filament"/>
-    </visual>
-    <collision>
-      <origin rpy="0 0 0" xyz="0 0 0"/>
-      <geometry>
-        <mesh filename="file://$(find thor_description)/meshes/art2.stl" scale="0.001 0.001 0.001"/>
-      </geometry>
-    </collision>
-  </link>
-  <joint name="joint_2" type="revolute">
-    <origin xyz="0 -0.0318752 0.0974304" rpy="1.5707963267948966 -1.5707963267948966 0"/>
-    <parent link="link_1"/>
-    <child link="link_2"/>
-    <axis xyz="0 0 1"/>
-    <limit lower="-0.4" upper="0.4" effort="4" velocity="1.1" />
-  </joint>
-  <!-- Блок Art 3 -->
-  <link name="link_3">
-    <inertial>
-      <origin rpy="0 0 0" xyz="-0.00029765 -0.023661 -0.0019125"/>
-      <mass value="0.1787"/>
-      <inertia ixx="0.0001685" ixy="-2.7713E-05" ixz="5.6885E-06" iyy="0.00012865" iyz="2.9256E-05" izz="0.00020744"/>
-    </inertial>
-    <visual>
-      <origin rpy="0 0 0" xyz="0 0 0"/>
-      <geometry>
-        <mesh filename="file://$(find thor_description)/meshes/art3.stl" scale="0.001 0.001 0.001"/>
-      </geometry>
-      <material name="filament"/>
-    </visual>
-    <collision>
-      <origin rpy="0 0 0" xyz="0 0 0"/>
-      <geometry>
-        <mesh filename="file://$(find thor_description)/meshes/art3.stl" scale="0.001 0.001 0.001"/>
-      </geometry>
-    </collision>
-  </link>
-  <joint name="joint_3" type="revolute">
-    <origin xyz="0.160 0 0" rpy="0 0 0"/>
-    <parent link="link_2"/>
-    <child link="link_3"/>
-    <axis xyz="0 0 -1"/>
-    <limit lower="-1" upper="1" effort="4" velocity="1.1" />
-  </joint>
-  <!-- Блок Art 4 -->
-  <link name="link_4">
-    <inertial>
-      <origin rpy="0 0 0" xyz="-0.0016798 -0.00057319 -0.074404"/>
-      <mass value="0.34936"/>
-      <inertia ixx="0.0030532" ixy="-1.8615E-05" ixz="-7.0047E-05" iyy="0.0031033" iyz="-2.3301E-05" izz="0.00022264"/>
-    </inertial>
-    <visual>
-      <origin rpy="0 0 0" xyz="0 0 0"/>
-      <geometry>
-        <mesh filename="file://$(find thor_description)/meshes/art4.stl" scale="0.001 0.001 0.001"/>
-      </geometry>
-      <material name="filament"/>
-    </visual>
-    <collision>
-      <origin rpy="0 0 0" xyz="0 0 0"/>
-      <geometry>
-        <mesh filename="file://$(find thor_description)/meshes/art4.stl" scale="0.001 0.001 0.001"/>
-      </geometry>
-    </collision>
-  </link>
-  <joint name="joint_4" type="revolute">
-    <origin xyz="0.0885 0 -0.035" rpy="0 1.5707963267948966 0"/>
-    <parent link="link_3"/>
-    <child link="link_4"/>
-    <axis xyz="0 0 1"/>
-    <limit lower="-3.1" upper="3.1" effort="4" velocity="1.1" />
-  </joint>
-  <!-- Блок Art 5 (наклон рабочего органа) -->
-  <link name="link_5">
-    <inertial>
-      <origin rpy="0 0 0" xyz="0.0015066 -1.3102E-05 -0.012585"/>
-      <mass value="0.11562"/>
-      <inertia ixx="5.5035E-05" ixy="-1.019E-08" ixz="-2.6243E-06" iyy="8.2921E-05" iyz="1.4437E-08" izz="5.2518E-05"/>
-    </inertial>
-    <visual>
-      <origin rpy="0 0 0" xyz="0 0 0"/>
-      <geometry>
-        <mesh filename="file://$(find thor_description)/meshes/art5.stl" scale="0.001 0.001 0.001"/>
-      </geometry>
-      <material name="filament"/>
-    </visual>
-    <collision>
-      <origin rpy="0 0 0" xyz="0 0 0"/>
-      <geometry>
-        <mesh filename="file://$(find thor_description)/meshes/art5.stl" scale="0.001 0.001 0.001"/>
-      </geometry>
-    </collision>
-  </link>
-  <joint name="joint_5" type="revolute">
-    <origin xyz="0 0 0.1" rpy="0 -1.5707963267948966 0"/>
-    <parent link="link_4"/>
-    <child link="link_5"/>
-    <axis xyz="0 0 -1"/>
-    <limit lower="-1.5" upper="1.5" effort="4" velocity="1" />
-  </joint>
-  <!-- Блок Art 6 (поворот рабочего органа) -->
-  <link name="link_6">
-    <inertial>
-      <origin rpy="0 0 0" xyz="2.9287E-10 -1.6472E-09 0.0091432"/>
-      <mass value="0.013863"/>
-      <inertia ixx="1.3596E-06" ixy="3.0585E-13" ixz="5.7102E-14" iyy="1.7157E-06" iyz="6.3369E-09" izz="2.4332E-06"/>
-    </inertial>
-    <visual>
-      <origin rpy="0 0 0" xyz="0 0 0"/>
-      <geometry>
-        <mesh filename="file://$(find thor_description)/meshes/art6.stl" scale="0.001 0.001 0.001"/>
-      </geometry>
-      <material name="filament"/>
-    </visual>
-    <collision>
-      <origin rpy="0 0 0" xyz="0 0 0"/>
-      <geometry>
-        <mesh filename="file://$(find thor_description)/meshes/art6.stl" scale="0.001 0.001 0.001"/>
-      </geometry>
-    </collision>
-  </link>
-  <joint name="joint_6" type="revolute">
-    <origin xyz="0 0 0" rpy="0 1.5707963267948966 0"/>
-    <parent link="link_5"/>
-    <child link="link_6"/>
-    <axis xyz="0 0 -1"/>
-    <limit lower="-3.1" upper="3.1" effort="4" velocity="1.1" />
-  </joint>
-  <!-- Материальная точка, конец кинематической цепи thor_manupulator -->
-  <link name="ee_link" />
-  <joint name="ee_joint" type="fixed">
-    <parent link="link_6" />
-    <child link="ee_link" />
-    <origin xyz="0 0 0.06" rpy="0 0 0" />
-  </joint>
-  <!-- ===============================================================-->
-  <!-- Клешня, кинематическая цепь thor_gripper -->
-  <!-- ===============================================================-->
-  <joint name="gripper_base_joint" type="fixed">
-      <origin xyz="-0.016 0.0 0.008" rpy="1.5708 0.0 1.5708"/>
-      <parent link="ee_link"/>
-      <child link="gripper_base_link"/>
-  </joint>
-  <!-- Основание захвата -->
-  <link name="gripper_base_link">
-      <collision>
-          <origin xyz="0 0 0" rpy="0 0 0" />
+      <parent link="world"/>
+      <child link="base_link" />
+    </joint>
+    <link name="base_link">
+      <inertial>
+        <origin rpy="0 0 0" xyz="-4.6941E-06 0.054174 0.038824"/>
+        <mass value="0.7102"/>
+        <inertia ixx="0.0039943" ixy="3.697E-07" ixz="-5.7364E-08" iyy="0.0014946" iyz="-0.00036051" izz="0.0042554"/>
+      </inertial>
+      <visual>
+        <origin rpy="0 0 0" xyz="0 0 0"/>
+        <geometry>
+          <mesh filename="file://$(find thor_description)/meshes/base.stl" scale="0.001 0.001 0.001" />
+        </geometry>
+        <material name="filament">
+          <color rgba="0.69803922 0.82352941 0.94117647 1.0"/>
+        </material>
+      </visual>
+      <collision>
+        <origin rpy="0 0 0" xyz="0 0 0"/>
+        <geometry>
+          <mesh filename="file://$(find thor_description)/meshes/base.stl" scale="0.001 0.001 0.001"/>
+        </geometry>
+      </collision>
+    </link>
+    <!-- Блок с электроникой -->
+    <joint name="box_joint" type="fixed">
+      <origin xyz="-0.1 0 0.025" rpy="0 0 0"/>
+      <parent link="base_link"/>
+      <child link="box_link"/>
+    </joint>
+    <link name="box_link">
+        <visual>
           <geometry>
-              <mesh filename="file://$(find thor_description)/meshes/hand.stl" scale="0.001 0.001 0.001" />
-          </geometry>
-      </collision>
-      <visual>
-          <origin xyz="0 0 0" rpy="0 0 0" />
-          <geometry>
-              <mesh filename="file://$(find thor_description)/meshes/hand.stl" scale="0.001 0.001 0.001" />
+            <box size="0.18 0.15 0.05"/>
           </geometry>
           <material name="filament"/>
-      </visual>
-      <inertial>
-          <mass value="0.11" />
-          <inertia ixx="17803724" iyy="21783168" izz="28014524" ixy="-414543.5" ixz="225471.4375" iyz="-1840743.875" />
-      </inertial>
-  </link>
-  <!-- Узлы пальцев, 1-ый узел ведущий, второй - ведомый (задается при помощи тега mimic) -->
-  <joint name="gripper_jaw1_joint" type="prismatic">
-      <parent link="gripper_base_link" />
-      <child link="gripper_jaw1_link" />
-      <origin rpy="0 0 0" xyz="0.05 0.02 0" />
-      <axis xyz="-0.5547 0.8321 0"/>
-      <limit effort="100" lower="0.0" upper="0.06" velocity="10" />
-      <dynamics damping="0.3" friction="0.5" />
-  </joint>
-  <joint name="gripper_jaw2_joint" type="prismatic">
-      <parent link="gripper_base_link" />
-      <child link="gripper_jaw2_link" />
-      <origin rpy="0 0 0" xyz="-0.05 0.02 0" />
-      <axis xyz="0.5547 0.8321 0"/>
-      <limit effort="100" lower="0.0" upper="0.06" velocity="10" />
-      <mimic joint="gripper_jaw1_joint" />
-      <dynamics damping="0.3" friction="0.5" />
-  </joint>
-  <!-- Пальцы -->
-  <link name="gripper_jaw1_link">
-      <collision>
-          <origin xyz="0 0 0" rpy="0 0 0" />
-          <geometry>
-              <mesh filename="file://$(find thor_description)/meshes/finger.stl" scale="-0.001 0.001 0.001" />
-          </geometry>
-      </collision>
-      <visual>
-          <origin xyz="0 0 0" rpy="0 0 0" />
-          <geometry>
-              <mesh filename="file://$(find thor_description)/meshes/finger.stl" scale="-0.001 0.001 0.001" />
-          </geometry>
-          <material name="filament"/>
-      </visual>
-      <inertial>
-          <mass value="0.01" />
-          <inertia ixx="3358780.25" iyy="627437.875" izz="3410634.5" ixy="-145110.265625" ixz="93.539124" iyz="1280.361816" />
-      </inertial>
-  </link>
-  <link name="gripper_jaw2_link">
-      <collision>
-          <origin xyz="0 0 0" rpy="0 0 0" />
-          <geometry>
-              <mesh filename="file://$(find thor_description)/meshes/finger.stl" scale="0.001 0.001 0.001" />
-          </geometry>
-      </collision>
-      <visual>
-          <origin xyz="0 0 0" rpy="0 0 0" />
-          <geometry>
-              <mesh filename="file://$(find thor_description)/meshes/finger.stl" scale="0.001 0.001 0.001" />
-          </geometry>
-          <material name="filament"/>
-      </visual>
-      <inertial>
-          <mass value="0.01" />
-          <inertia ixx="3358780.25" iyy="627437.875" izz="3410634.5" ixy="-145110.265625" ixz="93.539124" iyz="1280.361816" />
-      </inertial>
-  </link>
+        </visual>
+    </link>
+    <!-- <Блок Art 1 -->
+    <link name="link_1">
+      <inertial>
+        <origin rpy="0 0 0" xyz="-0.022706 0.04294 -0.12205"/>
+        <mass value="0.88065"/>
+        <inertia ixx="0.0034" ixy="0.00042296" ixz="-0.00089231" iyy="0.0041778" iyz="0.0010848" izz="0.0027077"/>
+      </inertial>
+      <visual>
+        <origin rpy="0 0 0" xyz="0 0 0"/>
+        <geometry>
+          <mesh filename="file://$(find thor_description)/meshes/art1.stl" scale="0.001 0.001 0.001"/>
+        </geometry>
+        <material name="filament"/>
+      </visual>
+      <collision>
+        <origin rpy="0 0 0" xyz="0 0 0"/>
+        <geometry>
+          <mesh filename="file://$(find thor_description)/meshes/art1.stl" scale="0.001 0.001 0.001"/>
+        </geometry>
+      </collision>
+    </link>
+    <joint name="joint_1" type="revolute">
+      <origin xyz="0 0 0.104" rpy="0 0 0"/>
+      <parent link="base_link"/>
+      <child link="link_1"/>
+      <axis xyz="0 0 1"/>
+      <limit lower="-1.5" upper="1.5" effort="4" velocity="1.1" />
+    </joint>
+    <!-- Блок Art 2 -->
+    <link name="link_2">
+      <inertial>
+        <origin rpy="0 0 0" xyz="0.064818 -0.11189 -0.038671"/>
+        <mass value="0.57738"/>
+        <inertia ixx="0.0047312" ixy="0.0022624" ixz="0.00032144" iyy="0.0020836" iyz="-0.00056569" izz="0.0056129"/>
+      </inertial>
+      <visual>
+        <origin rpy="0 0 0" xyz="0 0 0"/>
+        <geometry>
+          <mesh filename="file://$(find thor_description)/meshes/art2.stl" scale="0.001 0.001 0.001"/>
+        </geometry>
+        <material name="filament"/>
+      </visual>
+      <collision>
+        <origin rpy="0 0 0" xyz="0 0 0"/>
+        <geometry>
+          <mesh filename="file://$(find thor_description)/meshes/art2.stl" scale="0.001 0.001 0.001"/>
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
File: thor_hardware_interface/urdf/thor.urdf.xacro (robot description, xacro)
@@ -5,9 +5,8 @@
   <xacro:arg name="calibrate" default="True"/>
   <xacro:arg name="include_gripper" default="true"/>
-  <xacro:include filename="$(find thor_description)/urdf/thor_macro.xacro"/>
+  <xacro:include filename="$(find thor_description)/urdf/thor.urdf.xacro"/>
   <xacro:include filename="$(find thor_description)/urdf/thor.ros2_control.xacro"/>
   <link name="world" />
-  <xacro:thor_robot parent="world">
-    <origin xyz="0 0 0" rpy="0 0 0" />
+  <xacro:thor_robot>
   </xacro:thor_robot>
   <xacro:thor_ros2_control
