Commit message: Fix: два линка world.

File: thor_hardware_interface/urdf/thor.urdf.xacro (robot description, xacro)
@@ -7,5 +7,4 @@
   <xacro:include filename="$(find thor_description)/urdf/thor.urdf.xacro"/>
   <xacro:include filename="$(find thor_description)/urdf/thor.ros2_control.xacro"/>
-  <link name="world" />
   <xacro:thor_robot>
   </xacro:thor_robot>
